File: pcb/Telegraph.sch (KiCad schematic (older format))
At the start: 184 parts

Commit message: Proceeding with pcb
Parts:
- removed C? (x2): 10n, CAP_0603, symbol C
- removed D? (x6): LED, symbol LED
- removed D? (x2): SMBJ15CA, symbol DIODE_TVS
- removed Q? (x6): BC848, symbol NPN
- removed R? (x6): 4k7, RES_0603, symbol R
- removed R? (x8): 10k, RES_0603, symbol R
- removed R? (x6): 1k, RES_0603, symbol R
- removed R? (x2): 150, RES_0603, symbol R
- removed R? (x2): 20k, RES_0603, symbol R
- removed XL? (x2): CONN_2, symbol CONN_2
- added C16, C20, C51: 0.1u, Capacitors:CAP_0603, symbol C
- added C17: 1000u, Capacitors:CAP_10xxR, symbol CP
- added C18: 1000pF, Capacitors:CAP_0603, symbol C
- added C19: 1u, Capacitors:CAP_0603, symbol C
- added C21: 10u, Capacitors:CAP_0805, symbol C
- added D10, D27, D28, D3, D6: LED, LEDs:LED_Through-Hole-3mm, symbol LED
- added D13, D14: SS14, Diodes:SMA_DO214AC, symbol D_Shottky
- added D22: LED, LEDs:LED_0603, symbol LED
- added DA1: LP2951, SO_DIL_TSSOP:SO8, symbol LP2951
- added DA2: IPS6041, SO_DIL_TSSOP:SO8HEATSINK, symbol IPS6041
- added HOLE1, HOLE10, HOLE2, HOLE3, HOLE4, HOLE5, HOLE6, HOLE7, HOLE8, HOLE9: HOLE_METALLED, PCB:Hole3_5_out6mm, symbol HOLE_METALLED
- added L1: BLM, Inductors:IND_0402, symbol L
- added R2, R6: 4k7, Resistors:RES_0603, symbol R
- added R3, R72: 200, Resistors:RES_0603, symbol R
- added R51: 20k, Resistors:RES_0603, symbol R
- added R52: 12k, Resistors:RES_0603, symbol R
- added R55: 10k, Resistors:RES_0603, symbol R
- added R66, R73: 1k, Resistors:RES_0603, symbol R
- added R74: 330k, Resistors:RES_0603, symbol R
- added R75: 100k, Resistors:RES_0603, symbol R
- added SW1: DIPx4, BtnsSwitches:DIP_SMD_X4, symbol DIPx4
- added SW2: SWITCH_H, BtnsSwitches:SW_SS9, symbol SWITCH_H
- added SW4, SW5: SWITCH_2x, BtnsSwitches:BTN_PSM6, symbol SWITCH_2x
- added XL15: CONN_5, Connectors:PLS-5, symbol CONN_5
- added XL16, XL9: CONN_2, Connectors:TermiBlockHeader_508_x2_R, symbol CONN_2
- added XL8: BARREL_SOCKET, Connectors:Barrel, symbol BARREL_SOCKET
- BZ1: renamed from BZ?; footprint ~ -> Installation:BUZZER_HC0903
- C1, C2: renamed from C?; footprint Capacitors:CAP_0402 -> Capacitors:CAP_0603
- C10, C11, C12, C13, C14, C15, C8, C9: renamed from C?; footprint (none) -> Capacitors:CAP_0603
- C22, C23, C24, C25, C26, C27, C28, C29, C3, C30, C31, C36, C38, C4, C40, C41, C42, C43, C44, C45, C46, C47: renamed from C?; footprint CAP_0603 -> Capacitors:CAP_0603
- C32, C34, C50: renamed from C?; footprint CAP_0805 -> Capacitors:CAP_0805
- C33, C35: renamed from C?; footprint ~ -> Capacitors:CAP_0805
- C37, C39: renamed from C?; footprint CAP_1206 -> Capacitors:CAP_0603
- C48, C49: renamed from C?; footprint ~ -> Capacitors:CAP_10xxR
- C7: renamed from C?; footprint (none) -> Capacitors:CAP_0805
- D1, D2: renamed from D?; footprint (none) -> Diodes:SMB_DO214AA
- D15, D16, D17, D5, D9: renamed from D?; footprint (none) -> LEDs:LED_Through-Hole-3mm
- D18, D19, D20, D21: renamed from D?; footprint ~ -> LEDs:LED_0603
- D23, D24, D25, D26: renamed from D?; footprint ~ -> Diodes:SOD80C
- DD1: renamed from DD?; footprint (none) -> LQFP_TQFP:LQFP64
- Q1, Q10, Q11, Q2, Q6, Q7: renamed from Q?; footprint (none) -> SOT:SOT23-3
- Q14: renamed from Q?; footprint ~ -> SOT:SOT23-3
- R1, R10, R13, R14, R18, R19, R22, R23, R26, R27, R28, R29, R34, R35, R38, R39, R42, R43, R5, R53, R54, R56, R57, R58, R59, R60, R61, R62, R63, R64, R65, R67, R68, R69, R70, R71, R9: renamed from R?; footprint RES_0603 -> Resistors:RES_0603
- R17: renamed from R?; footprint Resistors:RES_0402 -> Resistors:RES_0603
- R46, R47, R48, R49, R50: renamed from R?; footprint (none) -> Resistors:RES_0603
- SW3: renamed from SW?; footprint (none) -> BtnsSwitches:BTN_6x6
- TP1, TP10, TP11, TP12, TP13, TP14, TP2, TP3, TP4, TP5, TP6, TP7, TP8, TP9: renamed from TP?; footprint (none) -> PCB:TESTPOINT_1MM
- U1, U2: renamed from U?; footprint ~ -> SO_DIL_TSSOP:HTSSOP28
- VCap1, VCap2: renamed from VCap?; footprint (none) -> Capacitors:CAP_0603
- XL1, XL2: renamed from XL?; footprint (none) -> Connectors:SPRING_TERM_XY124V_A_2
- XL10, XL11, XL12, XL13, XL14: renamed from XL?; footprint (none) -> Connectors:PLS-2
- XL17, XL18: renamed from XL?; footprint ~ -> Connectors:TermiBlockHeader_508_x4_R
- XL5: renamed from XL?; footprint ~ -> Connectors:PLS-3
- XL6: renamed from XL?; footprint ~ -> Connectors:PLS-4
- XTAL1: renamed from XTAL?; footprint CRYSTAL -> Quartz:0503x4-4
- gave numbers to parts that had none: 2
Connections:
- net +5V is gone; now on net +3.3V: BZ1.2, C50.1
- net TrgOut3 is gone; now on net LED1: DD1.16 ((ADC123-2)/T5C3/T9C1/T2C3/TX2/PA2)
- net TrgOut4 is gone; now on net LED2: DD1.17 ((ADC123-3)/T5C4/T9C2/T2C4/RX2/PA3)
- net USB_DM is gone; now on net D-: DD1.44 (OTGFS_DM/T1C4/PA11)
- net USB_DP is gone; now on net D+: DD1.45 (OTGFS_DP/PA12)
- net +12V: now also C16.1, C17.1, C20.1, C21.1, DA1.8 (In), DA2.5 (Vcc), DA2.6 (Vcc), DA2.7 (Vcc), DA2.8 (Vcc), R66.1, SW2.1
- net +3.3V: now also C18.1, C19.1, DA1.1 (Out), L1.2, R51.1; no longer C14.1, DD1.13 (VDDA)
- net BUSY/SYNC_1: now also DD1.8 ((ADC123-10)/PC0)
- net BUSY/SYNC_2: now also DD1.11 ((ADC123-13)/MOSI2/PC3)
- net FLAG_1: now also DD1.10 ((ADC123-12)/MISO2/PC2)
- net FLAG_2: now also DD1.25 ((ADC12-15)/PC5)
- net GND: now also C16.2, C17.2, C19.2, C20.2, C21.2, C51.2, D10.A, D27.C, D28.C, D3.C, D6.C, DA1.3 (Shdn), DA1.4 (GND), DA2.1 (GND), HOLE1.H, HOLE10.H, HOLE2.H, HOLE3.H, HOLE4.H, HOLE5.H, HOLE6.H, HOLE7.H, HOLE8.H, HOLE9.H, R52.2, R75.1, SW1.1, SW1.2, SW1.3, SW1.4, SW2.H, XL15.5, XL16.2 (PM), XL8.GND, XL9.2 (PM)
- net GPIO1: now also DD1.40 (MCO2/T8C4/SDA3/T3C4/SDIO_D1/PC9)
- net GPIO2: now also DD1.51 (SCK3/TX4/TX3/SDIO_D2/PC10)
- net GPIO3: now also DD1.52 (MISO3/RX4/RX3/SDIO_D3/PC11)
- net GPIO4: now also DD1.53 (MOSI3/TX5/CK3/SDIO_CK/PC12)
- net LineIn1: now also SW4.2, SW4.5; no longer Q1.3 (C), R1.1, R13.2, R18.1, R5.1
- net LineIn2: now also SW5.2, SW5.5; no longer Q2.3 (C), R14.2, R19.1
- net OUT1_1A: now also XL17.2 (PM); no longer XL17.1 (P1)
- net OUT1_2A: now also XL17.1 (P1); no longer XL17.2 (PM)
- net OUT2_1A: now also XL18.2 (PM); no longer XL18.1 (P1)
- net OUT2_2A: now also XL18.1 (P1); no longer XL18.2 (PM)
- net STBY/RST: now also DD1.37 (T8C1/TX6/T3C1/SDIO_D6/PC6)
- net SW_1: now also DD1.9 ((ADC123-11)/PC1)
- net SW_2: now also DD1.24 ((ADC12-14)/PC4)
- net LED3: now reaches R49.1
- net LED3: now also DD1.50 (PA15)
- net LED2: now reaches R48.1
- net LED1: now reaches R47.1
- net LED4: now reaches DD1.2 (PC13)
- net LED4: now also R72.1
- net DS3: now reaches DD1.29 (PB10/SCK2/SCL2/TX3/T2C3)
- net DS3: now also SW1.6
- net DS4: now reaches DD1.30 (PB11/SDA2/RX3/T2C4)
- net DS4: now also SW1.5
- net RSL1: now reaches DD1.33 (PB12/CK3)
- net RSL1: now also XL15.1
- net RSL2: now reaches DD1.34 (PB13/SCK2)
- net RSL2: now also XL15.2
- net RSL3: now reaches DD1.35 (PB14/MISO2/T12C1)
- net RSL3: now also XL15.3
- net RSL4: now reaches DD1.36 (PB15/MOSI2/T12C2)
- net RSL4: now also XL15.4
- net DS1: now reaches DD1.38 (T8C2/RX6/T3C2/SDIO_D7/PC7)
- net DS1: now also SW1.8
- net DS2: now reaches DD1.39 (T8C3/T3C3/CK6/SDIO_D0/PC8)
- net DS2: now also SW1.7
- net MagnetIN: now reaches DD1.43 (OTGFS_ID/T1C3/RX1/PA10)
- net MagnetIN: now also R55.1
- net LineTx3 renamed BatteryMeas
- net BatteryMeas: now also C51.1, R74.1, R75.2
- net LineTx4 renamed LED_BT
- net LED_BT: now also R3.1
- net SDI_3: no longer names the net of U2.18 (SDO)
- new net: Q1.3 (C), R13.2, R18.1, SW4.1, SW4.6
- new net: R1.1, R5.1, SW4.3, SW4.4
- new net: Q2.3 (C), R14.2, R19.1, SW5.1, SW5.6
- new net: C14.1, DD1.13 (VDDA), L1.1
- new net: C18.2, DA1.7 (Feedback), R51.2, R52.1
- new net: D28.A, R73.2
- new net: DA2.2 (Input), R55.2
- new net: D22.C, DA2.3 (Diag)
- new net: D22.A, R66.2
- new net: R2.1, R6.1, SW5.3, SW5.4
- new net: D6.A, R2.2
- new net: D10.C, R6.2
- new net: D27.A, R72.2
- new net: D3.A, R3.2
- new net MagnetOUT: DA2.4 (Out), XL16.1 (P1)
- new net PWR_BAT: D14.A, R74.2, XL9.1 (P1)
- new net PWR_IN: D13.C, D14.C, SW2.2
- new net PWR_SRC: D13.A, R73.1, XL8.PWR
- no-connect marks 22 -> 15
Other:
- note added: "Battery Low"
- note added: "Maybe\nLimiters"
- note added: "Periphery\n\nUART1 (PB6, PB7) = Debug UART\n\nTIM1 C3 = MagnetIN\nTIM2 C2 = Buzzer\nTIM3 C1,C2 = LineTx1...4\nTIM10 C1 = STEP_CLK_1\nTIM11 C1 = STEP_CLK_2\n\nADC 0,1 (PA0,PA1) = line inputs\nADC 8 (PB0) = Battery measurement"
- note added: "Rotary\nSwitch"
- note removed: "Line 3"
- note removed: "Line 4"
- note removed: "Periphery\n\nUART1 (PB6, PB7) = Debug UART\n\nTIM2 C2 = Buzzer\nTIM3 C1...C4 = LineTx1...4\nTIM10C1 = STEP_CLK_1\nTIM11C1 = STEP_CLK_2\n\nADC 0...3 (PA0...PA3) = line inputs"
- moved on the sheet: C11, C12, C7, C8, C9, D15, D16, D17, D5, D9, R1, R47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

Commit message: Pcb routing started
Parts:
- removed D28: LED, LEDs:LED_Through-Hole-3mm, symbol LED
- removed HOLE7: HOLE_METALLED, PCB:Hole3_5_out6mm, symbol HOLE_METALLED
- removed R2, R5: 4k7, Resistors:RES_0603, symbol R
- added D4, D7: LED, LEDs:LED_Through-Hole-3mm, symbol LED
- added R4, R7: 200, Resistors:RES_0603, symbol R
- R73: value 1k -> 10k
Connections:
- net DS1: now also DD1.29 (PB10/SCK2/SCL2/TX3/T2C3); no longer DD1.38 (T8C2/RX6/T3C2/SDIO_D7/PC7)
- net DS2: now also DD1.30 (PB11/SDA2/RX3/T2C4); no longer DD1.39 (T8C3/T3C3/CK6/SDIO_D0/PC8)
- net DS3: now also DD1.38 (T8C2/RX6/T3C2/SDIO_D7/PC7); no longer DD1.29 (PB10/SCK2/SCL2/TX3/T2C3)
- net DS4: now also DD1.39 (T8C3/T3C3/CK6/SDIO_D0/PC8); no longer DD1.30 (PB11/SDA2/RX3/T2C4)
- net GND: now also D4.C, D7.C
- net at D5.A, R1.2: now also D9.C
- net LED_BT_LOW: now reaches DD1.28 (PB2/BOOT1)
- net LED_BT_LOW: now also R4.1
- net PwrSrcSns: now reaches DD1.3 ((OC32IN)/PC14)
- net PwrSrcSns: now also R73.2
- net LED_SRC_PWR: now reaches DD1.4 ((OC32OUT)/PC15)
- net LED_SRC_PWR: now also R7.1
- net at D6.A: now also D10.C, R6.2
- net LED_BT renamed LED_BT_PWR
- new net: D4.A, R4.2
- new net: D7.A, R7.2
- no-connect marks 15 -> 12
Other:
- note added: "Battery Pwr"
- note added: "Source Pwr"
- moved on the sheet: D3, R1, R3, R6

Commit message: Proceeding with pcb
Parts:
- removed C31: 100p, Capacitors:CAP_0603, symbol C
- removed R65: 39K, Resistors:RES_0603, symbol R
Connections:
- net MOTOR_MISO: now also U2.18 (SDO)
- no-connect marks 12 -> 11
Changed lines of the file:
@@
 $EndComp
 $Comp
-L R R65
-U 1 1 55A679C5
-P 17250 7900
-F 0 "R65" V 17330 7750 50  0000 C CNN
-F 1 "39K" V 17250 7900 50  0000 C CNN
-F 2 "Resistors:RES_0603" V 17330 8000 28  0000 C CNN
-F 3 "~" H 17250 7900 60  0000 C CNN
-	1    17250 7900
-	1    0    0    -1
-$EndComp
-$Comp
 L C C23
 U 1 1 55A679CC
@@
 	1    0    0    -1
 $EndComp
-$Comp
-L C C31
-U 1 1 55A679D3
-P 17250 9250
-F 0 "C31" H 17150 9150 50  0000 L CNN
-F 1 "100p" H 17150 9350 50  0000 L CNN
-F 2 "Capacitors:CAP_0603" V 17350 9100 28  0000 C BNN
-F 3 "~" H 17250 9250 60  0000 C CNN
-	1    17250 9250
-	1    0    0    -1
-$EndComp
 Text Label 16600 8200 2    60   ~ 0
 STEP_CLK_2
@@
 $EndComp
 $Comp
-L GND #PWR050
-U 1 1 55A679F5
-P 17250 9600
-F 0 "#PWR050" H 17340 9580 30  0001 C CNN
-F 1 "GND" H 17250 9520 30  0001 C CNN
-F 2 "" H 17250 9600 60  0000 C CNN
-F 3 "" H 17250 9600 60  0000 C CNN
-	1    17250 9600
-	1    0    0    -1
-$EndComp
-$Comp
 L LED D21
 U 1 1 55A679FB
@@
 Text Label 13000 4050 2    60   ~ 0
 DS4
-NoConn ~ 17650 9000
 $Comp
 L PWR_FLAG #FLG0110
@@
 Wire Wire Line
 	19650 8100 20250 8100
-Wire Wire Line
-	17250 8150 17250 9050
-Connection ~ 17250 8300
 Connection ~ 17000 8400
 Wire Wire Line
@@
 	17000 8150 17000 9050
 Wire Wire Line
-	17250 9600 17250 9450
-Wire Wire Line
 	17000 9450 17000 9600
 Wire Wire Line
 	16750 9450 16750 9600
 Wire Wire Line
-	16750 7550 17250 7550
-Wire Wire Line
-	17250 7550 17250 7650
-Connection ~ 17000 7550
-Wire Wire Line
 	15650 6800 15650 6700
 Wire Wire Line
@@
 Wire Wire Line
 	10800 5300 10800 5200
-Connection ~ 10800 5300
 Wire Wire Line
 	8050 5200 8050 5350
@@
 Wire Wire Line
 	17250 14150 17150 14150
+Text Label 17550 9000 2    60   ~ 0
+MOTOR_MISO
+Wire Wire Line
+	17550 9000 17650 9000
+Wire Wire Line
+	17000 7550 16750 7550
 $EndSCHEMATC
