File: pcb/Telegraph.kicad_pcb (KiCad board)
At the start: 2 copper layers, 189 parts, among them Q1 BC848, Q10 BC848, Q11 BC848, Q14 MMBT2222, Q2 BC848, Q5 DVIUC6-4SC6, Q6 BC848, Q7 BC848, SW1 DIPx4, SW2 SWITCH_H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

Commit message: Pcb routing started
Parts:
- removed D28: LED, LEDs:LED_Through-Hole-3mm
- removed HOLE7: HOLE_METALLED, PCB:Hole3_5_out6mm
- removed R2, R5: 4k7, Resistors:RES_0603
- added D4: LED, LEDs:LED_Through-Hole-3mm, F.Cu at (144.0, 31.0)
- added D7: LED, LEDs:LED_Through-Hole-3mm, F.Cu at (131.0, 31.0)
- added R4: 200, Resistors:RES_0603, F.Cu at (143.6, 35.0)
- added R7: 200, Resistors:RES_0603, F.Cu at (130.6, 35.0)
- C28, C29, C34, C35, C38, C39, C41, C43, C45, C47, D24, D26, R68, R69, R70, R71: moved to B.Cu
- R73: value 1k -> 10k
- moved R17 211.5 mm to (77.0, 74.4), turned to 90 degrees
- moved C1 208.2 mm to (78.6, 74.4), turned to 90 degrees
- moved R73 202.6 mm to (81.6, 106.4), turned to 180 degrees
- moved R47 200.6 mm to (82.0, 31.0), turned to 180 degrees
- moved C19 199.0 mm to (96.6, 88.7), turned to 270 degrees
- moved R75 198.8 mm to (89.8, 101.8)
- moved R51 198.6 mm to (93.8, 87.9), turned to 180 degrees
- moved R18 197.3 mm to (93.6, 37.2)
- moved R6 195.9 mm to (88.0, 63.0)
- moved R27 194.0 mm to (98.8, 42.4), turned to 270 degrees
- moved R38 193.1 mm to (101.2, 34.4), turned to 90 degrees
- moved R55 192.4 mm to (94.0, 102.6), turned to 270 degrees
- moved Q5 192.1 mm to (84.0, 77.2), turned to 270 degrees
- moved R52 191.6 mm to (93.8, 91.1)
- moved C2 190.1 mm to (80.2, 74.4), turned to 270 degrees
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Connections:
- net /LED_BT renamed /LED_BT_PWR
- D6 pad A: Net-(D6-PadA) -> Net-(D10-PadC)
- D9 pad C: Net-(D9-PadC) -> Net-(D5-PadA)
- DD1 pad 28: (no net) -> /LED_BT_LOW
- DD1 pad 29: /DS3 -> /DS1
- DD1 pad 3: (no net) -> /PwrSrcSns
- DD1 pad 30: /DS4 -> /DS2
- DD1 pad 38: /DS1 -> /DS3
- DD1 pad 39: /DS2 -> /DS4
- DD1 pad 4: (no net) -> /LED_SRC_PWR
- R73 pad 2: Net-(D28-PadA) -> /PwrSrcSns
Other:
- board outline added: 87 x 88 mm
- net class Default: trace_width 0.25 -> 0.2; via_dia 0.6 -> 0.8; via_drill 0.4 -> 0.3
- net class Wide added: clearance 0.2, trace_width 0.5, via_dia 1, via_drill 0.5

Commit message: Proceeding with pcb
Parts:
- removed C31: 100p, Capacitors:CAP_0603
- removed R65: 39K, Resistors:RES_0603
- moved C8 28.1 mm to (133.4, 76.3), turned to 270 degrees
- moved VCap1 26.8 mm to (131.8, 76.3), turned to 270 degrees
- moved C13 25.9 mm to (115.6, 71.1), turned to 180 degrees
- moved C12 24.8 mm to (125.6, 76.3), turned to 270 degrees
- moved SW3 23.2 mm to (122.6, 53.1), turned to 180 degrees
- moved XTAL1 22.8 mm to (115.4, 66.9), turned to 270 degrees
- moved C9 22.1 mm to (137.6, 62.1), turned to 0 degrees
- moved VCap2 21.8 mm to (137.6, 63.7), turned to 0 degrees
- moved C10 21.7 mm to (115.6, 62.7), turned to 0 degrees
- moved L1 21.3 mm to (118.2, 70.7), turned to 270 degrees
- moved C14 19.8 mm to (119.6, 71.1), turned to 270 degrees
- moved R46 16.7 mm to (118.6, 66.9), turned to 270 degrees
- moved C15 15.1 mm to (119.6, 61.3), turned to 180 degrees
- moved C11 13.0 mm to (123.3, 58.3), turned to 90 degrees
- moved R50 11.8 mm to (125.8, 58.1), turned to 180 degrees
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Connections:
- U2 pad 18: (no net) -> /MOTOR_MISO
Routing:
- net GND: track 0.00 -> 698.5 mm, vias 0 -> 23
- net +12V: track 0.00 -> 229.9 mm, vias 0 -> 9
- net +3.3V: track 0.00 -> 216.1 mm, vias 0 -> 9
- net /D+: track 0.00 -> 72.7 mm, vias 0 -> 2
- net /D-: track 0.00 -> 72.5 mm, vias 0 -> 2
- net /PwrSrcSns: track 0.00 -> 70.1 mm, vias 0 -> 2
- net /STBY/RST: track 0.00 -> 68.7 mm, vias 0 -> 6
- net /LED1: track 0.00 -> 61.1 mm, vias 0 -> 2
- net /MagnetIN: track 0.00 -> 57.1 mm, vias 0 -> 2
- net /BatteryMeas: track 0.00 -> 56.2 mm, vias 0 -> 2
- net /LED2: track 0.00 -> 54.4 mm, vias 0 -> 2
- net Net-(DD1-Pad42): track 0.00 -> 52.0 mm, vias 0 -> 2
- net /TrgOut1: track 0.00 -> 43.5 mm, vias 0 -> 2
- net /MOTOR_CS: track 0.00 -> 43.1 mm, vias 0 -> 4
- net /LineTx2: track 0.00 -> 41.4 mm, vias 0 -> 2
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
Commit message: Proceeding
Routing:
- net /Vdd2: track 17.9 -> 45.3 mm, vias 2 -> 4
- net GND: track 698.5 -> 707.9 mm, vias 23 -> 24
- net +12V: track 229.9 -> 235.4 mm, vias 9 -> 12
- net /MOTOR_CS: track 43.1 -> 38.9 mm
- net /D-: track 72.5 -> 69.2 mm
- net /STBY/RST: track 68.7 -> 65.9 mm
- net /D+: track 72.7 -> 70.0 mm
- net /OUT2_1B: track 11.8 -> 13.0 mm
- net /OUT2_1A: track 11.6 -> 12.4 mm
- net /PwrSrcSns: track 70.1 -> 69.5 mm
- net /OUT2_2B: track 17.1 -> 17.7 mm
- net /DS2: track 32.4 -> 31.8 mm
- net /BUSY/SYNC_1: track 15.4 -> 14.9 mm
Other:
- net class Wide: via_dia 1 -> 0.9; via_drill 0.5 -> 0.4

Commit message: PCB sent to production
Parts:
- moved SW1 1.60 mm to (116.0, 40.4)
- moved C39 1.20 mm to (139.2, 103.8)
- moved HOLE6 1.00 mm to (105.0, 96.0)
- moved C37 0.80 mm to (116.8, 103.8)
Routing:
- net GND: track 707.9 -> 1506.7 mm, vias 24 -> 210
- net /MOTOR_SCK: track 14.4 -> 53.4 mm, vias 0 -> 3
- net /BUSY/SYNC_2: track 11.2 -> 48.4 mm, vias 0 -> 4
- net /SDI_2: track 0.00 -> 36.2 mm, vias 0 -> 3
- net /Vdd1: track 17.8 -> 51.6 mm, vias 2 -> 5
- net /FLAG_1: track 17.6 -> 45.6 mm, vias 2 -> 4
- net /MOTOR_CS: track 38.9 -> 63.3 mm, vias 4 -> 5
- net /FLAG_2: track 18.3 -> 41.4 mm, vias 2 -> 4
- net /BUSY/SYNC_1: track 14.9 -> 37.5 mm, vias 2 -> 4
- net /STBY/RST: track 65.9 -> 87.8 mm, vias 6 -> 8
- net /MOTOR_MISO: track 11.7 -> 33.4 mm, vias 0 -> 2
- net /SW_1: track 21.7 -> 42.4 mm, vias 2 -> 4
- net /MOTOR_MOSI: track 14.4 -> 33.2 mm
- net +12V: track 235.4 -> 251.9 mm, vias 12 -> 13
- net /SW_2: track 30.1 -> 44.9 mm
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- added copper zone on B.Cu, net GND
- added copper zone on F.Cu, net GND
Other:
- rule pad_to_mask_clearance: 0 -> 0.1
- board text added: "Key"
- board text added: "Line1"
- board text added: "Line2"
- board text added: "Magnet"
- board text added: "Motor1"
- board text added: "Motor2"
- board text added: "ON"
- board text added: "Quartz"
- board text added: "USB"
